File: ultrasonic_radar/circuit_design/circuit_design.kicad_pcb (KiCad board)
At the start: 2 copper layers, 11 parts

Commit message: circuit pcb design updated
Parts:
- added J1: Conn_01x02_Socket, Connector_Molex:Molex_KK-396_5273-02A_1x02_P3.96mm_Vertical, F.Cu at (138.0, 58.5)
- moved Ultrasonicsensor1-right1 59.8 mm to (114.9, 51.5), turned to 90 degrees
- moved Servo2-center1 41.0 mm to (92.5, 83.5), turned to 180 degrees
- moved Servo3-left1 38.4 mm to (79.5, 83.5), turned to 180 degrees
- moved Ultrasonicsensor3-left1 32.0 mm to (98.7, 51.5), turned to 90 degrees
- moved HW221-LEFT1 29.1 mm to (51.9, 56.0), turned to 90 degrees
- moved Ultrasonicsensor2-center1 28.7 mm to (84.4, 51.5)
- moved Servo1-right1 24.4 mm to (108.5, 83.5), turned to 180 degrees
- moved HW221-RIGHT1 23.9 mm to (74.9, 44.0), turned to -90 degrees
- moved Arduino-AnalogIO-A0toA8 12.4 mm to (113.2, 36.5)
Connections:
- Arduino-AnalogIO-A0toA8 pad 1: Pwm1-right -> RawEcho1
- Arduino-AnalogIO-A0toA8 pad 2: Pwm2-center -> RawEcho2
- Arduino-AnalogIO-A0toA8 pad 3: Pwm3-left -> RawEcho3
- Arduino-Pwm-0to7 pad 3: Pin_3 -> Pwm1-right
- Arduino-Pwm-0to7 pad 4: Pin_4 -> Pwm2-center
- Arduino-Pwm-0to7 pad 5: Pin_5 -> Pwm3-left
Routing:
- net +5V: track 0.00 -> 83.0 mm
- net GND: track 0.00 -> 68.1 mm
- net Pwm1-right: track 0.00 -> 49.2 mm
- net RawEcho2: track 0.00 -> 40.6 mm
- net Trigger2: track 0.00 -> 36.6 mm
- net Pwm2-center: track 0.00 -> 35.7 mm
- net Pwm3-left: track 0.00 -> 25.3 mm
- net RawEcho1: track 0.00 -> 22.0 mm
- net RawEcho3: track 0.00 -> 16.8 mm
